File: ICM-42688-P_breakout/ICM-42688-P_breakout.kicad_pcb (KiCad board)
At the start: 2 copper layers, 1 part, among them IC1 ICM-42688-P

Commit message: add schematic
add schematic
Parts:
- added C1: 0.01uF, Capacitor_SMD:C_0603_1608Metric, F.Cu at (134.0, 94.6)
- added C2: 0.1uF, Capacitor_SMD:C_0402_1005Metric, F.Cu at (138.4, 92.1)
- added C3: 22uF, Capacitor_SMD:C_0603_1608Metric, F.Cu at (138.4, 94.6)
- added J1: Conn_01x04_Female, Connector_PinHeader_2.54mm:PinHeader_1x04_P2.54mm_Vertical, F.Cu at (128.9, 94.6)
- added J2: Conn_01x04_Female, Connector_PinHeader_2.54mm:PinHeader_1x04_P2.54mm_Vertical, F.Cu at (142.9, 94.6)
Connections:
- IC1 pad 11: Net-(IC1-Pad11) -> Net-(C1-Pad2)
- IC1 pad 5: Net-(IC1-Pad5) -> Net-(C1-Pad1)
- IC1 pad 6: Net-(IC1-Pad6) -> Net-(C1-Pad2)
- IC1 pad 7: Net-(IC1-Pad7) -> Net-(C1-Pad2)
- IC1 pad 8: Net-(IC1-Pad8) -> Net-(C1-Pad1)

Commit message: 1st ordered to fusionPCB
1st ordered to fusionPCB
Routing:
- net Net-(C1-Pad2): track 0.00 -> 27.3 mm, vias 0 -> 3
- net Net-(C1-Pad1): track 0.00 -> 18.2 mm
- net Net-(IC1-Pad4): track 0.00 -> 12.4 mm, vias 0 -> 1
- net Net-(IC1-Pad13): track 0.00 -> 8.95 mm, vias 0 -> 1
- net Net-(IC1-Pad12): track 0.00 -> 8.59 mm
- net Net-(IC1-Pad14): track 0.00 -> 8.31 mm, vias 0 -> 1
- net Net-(IC1-Pad9): track 0.00 -> 7.22 mm, vias 0 -> 1
- net Net-(IC1-Pad1): track 0.00 -> 5.32 mm
- added copper zone on B.Cu, net Net-(C1-Pad2)
- added copper zone on F.Cu, net Net-(C1-Pad2)
Other:
- board outline added: 19 x 12.7 mm
- net class 0.5 added: clearance 0.2, trace_width 0.5, via_dia 0.8, via_drill 0.4
- net class 1.0 added: clearance 0.2, trace_width 1, via_dia 0.8, via_drill 0.4
- board text added: "CS INT2 INT2 GND"
- board text added: "SDO SDI SPC VDD"
